File: CardV1/CardV1.kicad_pcb (KiCad board)
At the start: 2 copper layers, 85.6 x 54 mm, 0 parts

Commit message: Almost Finish
Parts:
- added AE1: Antenna_Loop, CardV1:NFC-Antenna_6_79.24x47.62_0.6x0.6mm, F.Cu at (142.8, 73.0)
- added D1: LED, LED_SMD:LED_0603_1608Metric, F.Cu at (116.6, 79.2)
- added H1: GithubQRCode, CardV1:tingliangzhang-github-io, F.Cu at (163.8, 73.6)
- added J1: Conn_01x06_Male, Connector_PinHeader_2.54mm:PinHeader_1x06_P2.54mm_Vertical, F.Cu at (125.0, 87.0)
- added U1: M24LR04E-R, Package_SO:SO-8_3.9x4.9mm_P1.27mm, F.Cu at (116.5, 85.3)
Routing:
- net GND: track 0.00 -> 21.4 mm, vias 0 -> 2
- net Net-(AE1-Pad2): track 0.00 -> 17.2 mm, vias 0 -> 1
- net +5V: track 0.00 -> 14.7 mm
- net Net-(J1-Pad4): track 0.00 -> 7.55 mm
- net Net-(J1-Pad3): track 0.00 -> 7.02 mm
- net Net-(J1-Pad2): track 0.00 -> 6.49 mm
- net Net-(AE1-Pad1): track 0.00 -> 6.19 mm
- net Net-(J1-Pad1): track 0.00 -> 5.97 mm
- net (no net): vias 0 -> 1
Other:
- board text added: "Tina Zhang"
- board text added: "Tingliang Zhang Tsinghua University Tel 18141929603 E-mail ztl20@mails.tsinghua.edu.cn"

Commit message: Avatar
Parts:
- added G***: LOGO, CardV1:danni, B.Cu at (167.0, 81.3)
- added G***: LOGO, CardV1:cai, B.Cu at (115.0, 60.4)
- added G***: LOGO, CardV1:luna, B.Cu at (135.4, 60.7)
Other:
- board text added: "This is BMP Image Test"
