File: CardV2/CardV2.kicad_pcb (KiCad board)
At the start: 2 copper layers, 40 x 40 mm, 3 parts, among them U1 M24LR04E-R

Commit message: Almost Finish V2
Parts:
- added G***: LOGO, CardV2:NFClogo, F.Cu at (122.5, 82.5)
- moved D1 27.6 mm to (104.0, 98.0), turned to 180 degrees
- moved U1 20.4 mm to (104.0, 91.0), turned to 90 degrees
Routing:
- net Net-(AE1-Pad2): track 0.00 -> 13.3 mm, vias 0 -> 1
- net Net-(AE1-Pad1): track 0.00 -> 9.23 mm
- net Net-(D1-Pad1): track 0.00 -> 5.14 mm
- net Net-(D1-Pad2): track 0.00 -> 4.89 mm

Commit message: 失败的拼版
Parts:
- added G***: LOGO, CardV2:FutureLabLogo, B.Cu at (122.5, 82.5)
Other:
- board size 40 x 40 mm -> 95 x 100 mm
- board text added: "Designed By Zhang Tingliang"

Commit message: 拼板完成
Parts:
- moved G*** 3.54 mm to (120.0, 80.0)
Other:
- outline, holes or cut-outs redrawn
- board text removed: "Designed By Zhang Tingliang"
Changed lines of the file:
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@@
   (general
     (thickness 1.6)
-    (drawings 45)
+    (drawings 56)
     (tracks 17)
     (zones 0)
@@
       (outputformat 1)
       (mirror false)
-      (drillshape 1)
+      (drillshape 0)
       (scaleselection 1)
-      (outputdirectory ""))
+      (outputdirectory "CardV2Fab/"))
   )
   (net 0 "")
@@
   )
   (module CardV2:FutureLabLogo (layer B.Cu)
-    (at 122.5 82.5 180)
+    (at 120 80 180)
     (fp_text reference G*** (at 0 0) (layer B.SilkS) hide
       (effects (font (size 1.524 1.524) (thickness 0.3)) (justify mirror))
@@
     )
   )
-  (gr_line (start 95 145) (end 95 45) (layer Edge.Cuts) (width 0.05))
-  (gr_line (start 100 145) (end 95 145) (layer Edge.Cuts) (width 0.05))
-  (gr_line (start 100 55) (end 100 145) (layer Edge.Cuts) (width 0.05))
-  (gr_line (start 185 55) (end 100 55) (layer Edge.Cuts) (width 0.05))
-  (gr_line (start 185 145) (end 185 55) (layer Edge.Cuts) (width 0.05))
-  (gr_line (start 190 145) (end 185 145) (layer Edge.Cuts) (width 0.05))
-  (gr_line (start 190 45) (end 190 145) (layer Edge.Cuts) (width 0.05))
-  (gr_line (start 95 45) (end 190 45) (layer Edge.Cuts) (width 0.05))
+  (gr_line (start 185 62.5) (end 185 55) (layer Edge.Cuts) (width 0.05))
+  (gr_line (start 185 107.5) (end 185 97.5) (layer Edge.Cuts) (width 0.05))
+  (gr_line (start 185 145) (end 185 142.5) (layer Edge.Cuts) (width 0.05))
+  (gr_line (start 100 145) (end 100 142.5) (layer Edge.Cuts) (width 0.05))
+  (gr_line (start 100 97.5) (end 100 107.5) (layer Edge.Cuts) (width 0.05))
+  (gr_line (start 100 55) (end 100 62.5) (layer Edge.Cuts) (width 0.05))
+  (gr_line (start 140 130) (end 145 130) (layer Edge.Cuts) (width 0.05))
+  (gr_line (start 140 120) (end 145 120) (layer Edge.Cuts) (width 0.05))
+  (gr_line (start 170 100) (end 170 105) (layer Edge.Cuts) (width 0.05))
+  (gr_line (start 160 100) (end 160 105) (layer Edge.Cuts) (width 0.05))
+  (gr_line (start 140 75) (end 145 75) (layer Edge.Cuts) (width 0.05))
+  (gr_line (start 140 85) (end 145 85) (layer Edge.Cuts) (width 0.05))
+  (gr_line (start 125 100) (end 125 105) (layer Edge.Cuts) (width 0.05))
+  (gr_line (start 115 100) (end 115 105) (layer Edge.Cuts) (width 0.05))
+  (gr_line (start 190 45) (end 95 45) (layer Edge.Cuts) (width 0.05))
+  (gr_line (start 190 145) (end 190 45) (layer Edge.Cuts) (width 0.05))
+  (gr_line (start 185 145) (end 190 145) (layer Edge.Cuts) (width 0.05))
+  (gr_line (start 100 55) (end 185 55) (layer Edge.Cuts) (width 0.05))
+  (gr_line (start 95 145) (end 100 145) (layer Edge.Cuts) (width 0.05))
+  (gr_line (start 95 45) (end 95 145) (layer Edge.Cuts) (width 0.05))
   (gr_circle (center 149 109) (end 152 109) (layer Edge.Cuts) (width 0.05))
   (gr_arc (start 147.5 107.5) (end 147.5 105) (angle -90) (layer Edge.Cuts) (width 0.05))
@@
   (gr_line (start 147.5 145) (end 182.5 145) (layer Edge.Cuts) (width 0.05))
   (gr_line (start 145 107.5) (end 145 142.5) (layer Edge.Cuts) (width 0.05))
-  (gr_circle (center 149 64) (end 152 64) (layer Edge.Cuts) (width 0.05))
-  (gr_arc (start 147.5 62.5) (end 147.5 60) (angle -90) (layer Edge.Cuts) (width 0.05))
-  (gr_arc (start 182.5 62.5) (end 185 62.5) (angle -90) (layer Edge.Cuts) (width 0.05))
-  (gr_arc (start 182.5 97.5) (end 182.5 100) (angle -90) (layer Edge.Cuts) (width 0.05))
-  (gr_arc (start 147.5 97.5) (end 145 97.5) (angle -90) (layer Edge.Cuts) (width 0.05))
-  (gr_line (start 185 97.5) (end 185 62.5) (layer Edge.Cuts) (width 0.05))
-  (gr_line (start 182.5 60) (end 147.5 60) (layer Edge.Cuts) (width 0.05))
-  (gr_line (start 147.5 100) (end 182.5 100) (layer Edge.Cuts) (width 0.05))
-  (gr_line (start 145 62.5) (end 145 97.5) (layer Edge.Cuts) (width 0.05))
   (gr_circle (center 104 109) (end 107 109) (layer Edge.Cuts) (width 0.05))
   (gr_arc (start 102.5 107.5) (end 102.5 105) (angle -90) (layer Edge.Cuts) (width 0.05))
@@
   (gr_line (start 102.5 145) (end 137.5 145) (layer Edge.Cuts) (width 0.05))
   (gr_line (start 100 107.5) (end 100 142.5) (layer Edge.Cuts) (width 0.05))
-  (gr_text "Designed By Zhang Tingliang" (at 122.5 99) (layer F.SilkS)
-    (effects (font (size 1 1) (thickness 0.2)))
-  )
+  (gr_circle (center 149 64) (end 152 64) (layer Edge.Cuts) (width 0.05))
+  (gr_arc (start 147.5 62.5) (end 147.5 60) (angle -90) (layer Edge.Cuts) (width 0.05))
+  (gr_arc (start 182.5 62.5) (end 185 62.5) (angle -90) (layer Edge.Cuts) (width 0.05))
+  (gr_arc (start 182.5 97.5) (end 182.5 100) (angle -90) (layer Edge.Cuts) (width 0.05))
+  (gr_arc (start 147.5 97.5) (end 145 97.5) (angle -90) (layer Edge.Cuts) (width 0.05))
+  (gr_line (start 185 97.5) (end 185 62.5) (layer Edge.Cuts) (width 0.05))
+  (gr_line (start 182.5 60) (end 147.5 60) (layer Edge.Cuts) (width 0.05))
+  (gr_line (start 147.5 100) (end 182.5 100) (layer Edge.Cuts) (width 0.05))
+  (gr_line (start 145 62.5) (end 145 97.5) (layer Edge.Cuts) (width 0.05))
   (gr_line (start 100 62.5) (end 100 97.5) (layer Edge.Cuts) (width 0.05))
   (gr_line (start 137.5 60) (end 102.5 60) (layer Edge.Cuts) (width 0.05))
@@
   (segment (start 113.75 90.65) (end 103.36 90.65) (width 0.3) (layer B.Cu) (net 8))
   (segment (start 103.36 90.65) (end 103.36 90.65) (width 0.3) (layer B.Cu) (net 8))
-  (via blind (at 103.36 90.65) (size 0.5) (drill 0.3) (layers F.Cu B.Cu) (net 8))
+  (via (at 103.36 90.65) (size 0.5) (drill 0.3) (layers F.Cu B.Cu) (net 8) (status 1000000))
   (segment (start 103.365 90.655) (end 103.36 90.65) (width 0.3) (layer F.Cu) (net 8))
   (segment (start 103.365 93.575) (end 103.365 90.655) (width 0.3) (layer F.Cu) (net 8))

Commit message: 改为单板
Other:
- board size 95 x 100 mm -> 40 x 40 mm
- board text added: "Designed By Zhang Tingliang"
Changed lines of the file:
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@@
   (general
     (thickness 1.6)
-    (drawings 56)
+    (drawings 10)
     (tracks 17)
     (zones 0)
@@
     )
   )
-  (gr_line (start 185 62.5) (end 185 55) (layer Edge.Cuts) (width 0.05))
-  (gr_line (start 185 107.5) (end 185 97.5) (layer Edge.Cuts) (width 0.05))
-  (gr_line (start 185 145) (end 185 142.5) (layer Edge.Cuts) (width 0.05))
-  (gr_line (start 100 145) (end 100 142.5) (layer Edge.Cuts) (width 0.05))
-  (gr_line (start 100 97.5) (end 100 107.5) (layer Edge.Cuts) (width 0.05))
-  (gr_line (start 100 55) (end 100 62.5) (layer Edge.Cuts) (width 0.05))
-  (gr_line (start 140 130) (end 145 130) (layer Edge.Cuts) (width 0.05))
-  (gr_line (start 140 120) (end 145 120) (layer Edge.Cuts) (width 0.05))
-  (gr_line (start 170 100) (end 170 105) (layer Edge.Cuts) (width 0.05))
-  (gr_line (start 160 100) (end 160 105) (layer Edge.Cuts) (width 0.05))
-  (gr_line (start 140 75) (end 145 75) (layer Edge.Cuts) (width 0.05))
-  (gr_line (start 140 85) (end 145 85) (layer Edge.Cuts) (width 0.05))
-  (gr_line (start 125 100) (end 125 105) (layer Edge.Cuts) (width 0.05))
-  (gr_line (start 115 100) (end 115 105) (layer Edge.Cuts) (width 0.05))
-  (gr_line (start 190 45) (end 95 45) (layer Edge.Cuts) (width 0.05))
-  (gr_line (start 190 145) (end 190 45) (layer Edge.Cuts) (width 0.05))
-  (gr_line (start 185 145) (end 190 145) (layer Edge.Cuts) (width 0.05))
-  (gr_line (start 100 55) (end 185 55) (layer Edge.Cuts) (width 0.05))
-  (gr_line (start 95 145) (end 100 145) (layer Edge.Cuts) (width 0.05))
-  (gr_line (start 95 45) (end 95 145) (layer Edge.Cuts) (width 0.05))
-  (gr_circle (center 149 109) (end 152 109) (layer Edge.Cuts) (width 0.05))
-  (gr_arc (start 147.5 107.5) (end 147.5 105) (angle -90) (layer Edge.Cuts) (width 0.05))
-  (gr_arc (start 182.5 107.5) (end 185 107.5) (angle -90) (layer Edge.Cuts) (width 0.05))
-  (gr_arc (start 182.5 142.5) (end 182.5 145) (angle -90) (layer Edge.Cuts) (width 0.05))
-  (gr_arc (start 147.5 142.5) (end 145 142.5) (angle -90) (layer Edge.Cuts) (width 0.05))
-  (gr_line (start 185 142.5) (end 185 107.5) (layer Edge.Cuts) (width 0.05))
-  (gr_line (start 182.5 105) (end 147.5 105) (layer Edge.Cuts) (width 0.05))
-  (gr_line (start 147.5 145) (end 182.5 145) (layer Edge.Cuts) (width 0.05))
-  (gr_line (start 145 107.5) (end 145 142.5) (layer Edge.Cuts) (width 0.05))
-  (gr_circle (center 104 109) (end 107 109) (layer Edge.Cuts) (width 0.05))
-  (gr_arc (start 102.5 107.5) (end 102.5 105) (angle -90) (layer Edge.Cuts) (width 0.05))
-  (gr_arc (start 137.5 107.5) (end 140 107.5) (angle -90) (layer Edge.Cuts) (width 0.05))
-  (gr_arc (start 137.5 142.5) (end 137.5 145) (angle -90) (layer Edge.Cuts) (width 0.05))
-  (gr_arc (start 102.5 142.5) (end 100 142.5) (angle -90) (layer Edge.Cuts) (width 0.05))
-  (gr_line (start 140 142.5) (end 140 107.5) (layer Edge.Cuts) (width 0.05))
-  (gr_line (start 137.5 105) (end 102.5 105) (layer Edge.Cuts) (width 0.05))
-  (gr_line (start 102.5 145) (end 137.5 145) (layer Edge.Cuts) (width 0.05))
-  (gr_line (start 100 107.5) (end 100 142.5) (layer Edge.Cuts) (width 0.05))
-  (gr_circle (center 149 64) (end 152 64) (layer Edge.Cuts) (width 0.05))
-  (gr_arc (start 147.5 62.5) (end 147.5 60) (angle -90) (layer Edge.Cuts) (width 0.05))
-  (gr_arc (start 182.5 62.5) (end 185 62.5) (angle -90) (layer Edge.Cuts) (width 0.05))
-  (gr_arc (start 182.5 97.5) (end 182.5 100) (angle -90) (layer Edge.Cuts) (width 0.05))
-  (gr_arc (start 147.5 97.5) (end 145 97.5) (angle -90) (layer Edge.Cuts) (width 0.05))
-  (gr_line (start 185 97.5) (end 185 62.5) (layer Edge.Cuts) (width 0.05))
-  (gr_line (start 182.5 60) (end 147.5 60) (layer Edge.Cuts) (width 0.05))
-  (gr_line (start 147.5 100) (end 182.5 100) (layer Edge.Cuts) (width 0.05))
-  (gr_line (start 145 62.5) (end 145 97.5) (layer Edge.Cuts) (width 0.05))
+  (gr_text "Designed By Zhang Tingliang" (at 126 99) (layer F.SilkS)
+    (effects (font (size 1 1) (thickness 0.2)))
+  )
   (gr_line (start 100 62.5) (end 100 97.5) (layer Edge.Cuts) (width 0.05))
   (gr_line (start 137.5 60) (end 102.5 60) (layer Edge.Cuts) (width 0.05))
