File: CardV3/Card.kicad_pcb (KiCad board)
At the start: 2 copper layers, 85.6 x 54 mm, 6 parts, among them U1 M24LR04E-R, U2 P4080-BGA1295, U3 P4080-BGA1295

Commit message: V3 Update
Other:
- board text added: "Designed by Tingliang, Copyright © 2021 Tingliang Zhang CC BY-NC-ND"
- board text added: "Tingliang Zhang Tsinghua University 18141929603 ztl20@mails.tsinghua.edu.cn"
- board text removed: "Tingliang Zhang Tsinghua University Tel 18141929603 E-mail ztl20@mails.tsinghua.edu.cn"

Commit message: 我枯了，大家觉得这一版本不好看，改
Parts:
- added Linear_LGA-133: Linear_LGA-133_15.0x15.0mm_Layout12x12_P1.27mm, Package_LGA:Linear_LGA-133_15.0x15.0mm_Layout12x12_P1.27mm, B.Cu at (139.0, 85.0)
- added REF**: Inch_Ruler_3.5in_10, Card:Inch_Ruler_3.5in_10, B.Cu at (103.0, 100.0)
- added REF**: Resistor_Table_small, Card:Resistor_Table_small, B.Cu at (131.0, 73.0)
- added REF**: Metric_Ruler_90mm, Card:Metric_Ruler_90mm, B.Cu at (110.0, 50.0)
- added SO-24: SO-24_5.3x15mm_P1.27mm, Package_SO:SO-24_5.3x15mm_P1.27mm, B.Cu at (155.0, 85.0)
- LQFP-100_14x14mm: renamed from U3; value P4080-BGA1295 -> LQFP-100_14x14mm
- moved P4080-BGA1295 65.1 mm to (115.0, 86.0)
- moved LQFP-100_14x14mm 56.2 mm to (115.0, 60.0)
- renumbered U2 to P4080-BGA1295
Routing:
- net (no net): track 0.00 -> 129.4 mm
Other:
- board text added: "+10/50°C"
- board text added: "0.6A/1.2A"
- board text added: "0.75/30"
- board text added: "0.8A/1.5A"
- board text added: "0.9A/1.8A"
- board text added: "1.0/40"
- board text added: "1.0A/2.0A"
- board text added: "1.1A/2.3A"
- board text added: "1.2A/2.5A"
- board text added: "1.3/50"
- board text added: "1.4A/2.8A"
- board text added: "1.5/60"
- board text added: "1.5A/3.0A"
- board text added: "1.7A/3.4A"
- board text added: "1.9A/3.8A"
- board text added: "10/0.25"
- board text added: "12/0.30"
- board text added: "14/0.35"
- board text added: "16/0.40"
- board text added: "18/0.45"
- board text added: "1in=2.54cm 1cm≈0.394in 1mil=1/1000in 1mil=25,4µm"
- board text added: "2.0/80"
- board text added: "2.0A/4.0A"
- board text added: "2.1A/4.1A"
- board text added: "2.4A/4.9A"
- board text added: "20/0.50"
- board text added: "24/0.60"
- board text added: "28/0.70"
- board text added: "30/0.76"
- board text added: "32/0.80"
- board text added: "35µm=1.4mil"
- board text added: "40/1.00"
- board text added: "6/0.15"
- board text added: "8/0.20"
- board text added: "Font (mm/mil)"
- board text added: "mil/mm"
