File: CardV3.1/Card.kicad_pcb (KiCad board)
At the start: 2 copper layers, 85.6 x 54 mm, 11 parts, among them P4080-BGA1295 P4080-BGA1295, U1 M24LR04E-R

Commit message: V3.1
Parts:
- removed Linear_LGA-133: Linear_LGA-133_15.0x15.0mm_Layout12x12_P1.27mm, Package_LGA:Linear_LGA-133_15.0x15.0mm_Layout12x12_P1.27mm
- removed P4080-BGA1295: P4080-BGA1295, Package_BGA:BGA-256_17.0x17.0mm_Layout16x16_P1.0mm_Ball0.5mm_Pad0.4mm_NSMD
- removed the REF** at (131.0, 73.0)
- removed SO-24: SO-24_5.3x15mm_P1.27mm, Package_SO:SO-24_5.3x15mm_P1.27mm
- added G***: LOGO, Card:cai, F.Cu at (160.0, 60.0)
- AE1, D1, R1, U1: moved to B.Cu
- LQFP-100_14x14mm: moved to F.Cu
- moved U1 23.9 mm to (118.0, 62.0)
- moved R1 10.8 mm to (115.2, 70.7), turned to 180 degrees
- moved LQFP-100_14x14mm 10.0 mm to (125.0, 60.0), turned to 135 degrees
- moved D1 9.66 mm to (121.0, 70.6), turned to 180 degrees
Routing:
- net (no net): track 129.4 -> 36.8 mm
- net Net-(AE1-Pad2): track 0.00 -> 19.6 mm, vias 0 -> 2
- net GND: track 0.00 -> 13.4 mm
- net Net-(AE1-Pad1): track 0.00 -> 7.34 mm
- net +3V3: track 0.00 -> 7.20 mm
- net Net-(D1-Pad2): track 0.00 -> 4.23 mm
Other:
- board text added: "Just Another Geek"
- board text added: "Tingliang Zhang"
- board text added: "Tsinghua University Info Art Design"
- board text removed: "+10/50°C"
- board text removed: "0.6A/1.2A"
- board text removed: "0.75/30"
- board text removed: "0.8A/1.5A"
- board text removed: "0.9A/1.8A"
- board text removed: "1.0/40"
- board text removed: "1.0A/2.0A"
- board text removed: "1.1A/2.3A"
- board text removed: "1.2A/2.5A"
- board text removed: "1.3/50"
- board text removed: "1.4A/2.8A"
- board text removed: "1.5/60"
- board text removed: "1.5A/3.0A"
- board text removed: "1.7A/3.4A"
- board text removed: "1.9A/3.8A"
- board text removed: "10/0.25"
- board text removed: "12/0.30"
- board text removed: "14/0.35"
- board text removed: "16/0.40"
- board text removed: "18/0.45"
- board text removed: "1in=2.54cm 1cm≈0.394in 1mil=1/1000in 1mil=25,4µm"
- board text removed: "2.0/80"
- board text removed: "2.0A/4.0A"
- board text removed: "2.1A/4.1A"
- board text removed: "2.4A/4.9A"
- board text removed: "20/0.50"
- board text removed: "24/0.60"
- board text removed: "28/0.70"
- board text removed: "30/0.76"
- board text removed: "32/0.80"
- board text removed: "35µm=1.4mil"
- board text removed: "40/1.00"
- board text removed: "6/0.15"
- board text removed: "8/0.20"
- board text removed: "Font (mm/mil)"
- board text removed: "Tingliang Zhang Tsinghua University 18141929603 ztl20@mails.tsinghua.edu.cn"
- board text removed: "mil/mm"

Commit message: Finish 3.1 ?
Parts:
- removed LQFP-100_14x14mm: LQFP-100_14x14mm, Package_QFP:LQFP-100_14x14mm_P0.5mm
- removed REF**: Inch_Ruler_3.5in_10, Card:Inch_Ruler_3.5in_10
- removed REF**: Metric_Ruler_90mm, Card:Metric_Ruler_90mm
- added QR: https://interact.cool/, Card:interact.cool, F.Cu at (118.0, 66.0)
- moved G*** 16.4 mm to (150.0, 73.0)
Other:
- board text added: "Info Art Design Tsinghua University"
- board text removed: "Designed by Tingliang, Copyright © 2021 Tingliang Zhang CC BY-NC-ND"
- board text removed: "Tsinghua University Info Art Design"
