File: MassProduction/3任可欣/Card.kicad_pcb (KiCad board)
At the start: 2 copper layers, 85.6 x 54 mm, 7 parts, among them U1 M24LR04E-R

Commit message: 可欣
Other:
- board text added: "Fairy"
- board text removed: "Nefelibata"
