File: CardV4/Card.kicad_pcb (KiCad board)
At the start: 2 copper layers, 40 x 40 mm, 5 parts, among them U1 M24LR04E-R

Commit message: Finish and Print V4
Parts:
- removed D1: LED, LED_SMD:LED_0603_1608Metric
- removed the G*** at (120.0, 80.0)
- removed the G*** at (122.5, 82.5)
- added G***: LOGO, Card:FutureInteraction, B.Cu at (165.0, 82.5)
- AE1: footprint CardV2:NFC-Antenna_11_30.0x30.0_0.3x0.3mm -> Card:NFC-Antenna_13_25.0x25.0_0.3x0.2mm
- moved U1 63.1 mm to (167.0, 87.0)
- moved AE1 44.7 mm to (167.0, 87.0)
Routing:
- net Net-(U1-Pad4): track 5.14 -> 0.00 mm
- net Net-(U1-Pad1): track 4.89 -> 0.00 mm
- net Net-(AE1-Pad2): track 13.3 -> 16.9 mm, vias 1 -> 2
- net Net-(AE1-Pad1): track 9.23 -> 8.35 mm
Other:
- board size 40 x 40 mm -> 100 x 90 mm
- board text added: "Future Interaction Interest Group"
